Commit message: add new world

File: catkin_ws/src/husky/husky_description/urdf/accessories/camera.urdf.xacro (robot description, xacro)
@@ -30,7 +30,7 @@
     <!-- Add mesh for kinect -->
     <link name="${name}_link">
-      <origin xyz="0 0 0" rpy="0 0 0"/>
+      <!--origin xyz="0 0 0" rpy="0 0 0"/-->
       <visual>
-        <origin xyz="0 0 0" rpy="0 0 0"/>
+        <origin xyz="0 0 0" rpy="0 0 1.57"/>
         <geometry>
           <mesh filename="package://husky_description/meshes/accessories/kinect.dae" />

File: catkin_ws/src/husky/husky_description/urdf/accessories/velodyne_lidar.urdf.xacro (robot description, xacro)
@@ -2,5 +2,5 @@
 <robot xmlns:xacro="http://www.ros.org/wiki/xacro" name="VLP16_lidar">
   <xacro:property name="M_PI" value="3.1415926535897931" />
-  <xacro:macro name="VLP16_lidar" params="*origin parent:=base_link name:=velodyne topic:=/velodyne_points hz:=10 lasers:=16 samples:=2187 collision_range:=0.3 min_range:=0.5 max_range:=60.0 noise:=0.01 min_angle:=-${M_PI} max_angle:=${M_PI} gpu:=true">
+  <xacro:macro name="VLP16_lidar" params="*origin parent:=base_link name:=velodyne topic:=/velodyne_points hz:=10 lasers:=16 samples:=1875 collision_range:=0.3 min_range:=0.9 max_range:=130.0 noise:=0.008 min_angle:=-${M_PI} max_angle:=${M_PI} gpu:=true">
     <joint name="${name}_base_mount_joint" type="fixed">
       <xacro:insert_block name="origin" />
@@ -10,24 +10,29 @@
     <link name="${name}_base_link">
       <inertial>
-        <mass value="1.0"/>
-        <origin xyz="0 0 0.07212"/>
-        <inertia ixx="${(1.0 * (3.0*0.04267*0.04267 + 0.14424*0.14424)) / 12.0}" ixy="0" ixz="0"
-          iyy="${(1.0 * (3.0*0.04267*0.04267 + 0.14424*0.14424)) / 12.0}" iyz="0"
-          izz="${0.5 * 1.0 * (0.04267*0.04267)}"/>
+        <mass value="0.83"/>
+        <origin xyz="0 0 0.03585"/>
+        <inertia ixx="${(0.83 * (3.0*0.0516*0.0516 + 0.0717*0.0717)) / 12.0}" ixy="0" ixz="0"
+          iyy="${(0.83 * (3.0*0.0516*0.0516 + 0.0717*0.0717)) / 12.0}" iyz="0"
+          izz="${0.5 * 0.83 * (0.0516*0.0516)}"/>
       </inertial>
       <visual>
         <geometry>
-          <mesh filename="package://husky_description/meshes/accessories/HDL32E_base.dae" />
+          <mesh filename="package://velodyne_description/meshes/VLP16_base_1.dae" />
+        </geometry>
+      </visual>
+      <visual>
+        <geometry>
+          <mesh filename="package://velodyne_description/meshes/VLP16_base_2.dae" />
         </geometry>
       </visual>
       <collision>
-        <origin rpy="0 0 0" xyz="0 0 0.07212"/>
+        <origin rpy="0 0 0" xyz="0 0 0.03585"/>
         <geometry>
-          <cylinder radius="0.04267" length="0.14424"/>
+          <cylinder radius="0.0516" length="0.0717"/>
         </geometry>
       </collision>
     </link>
     <joint name="${name}_base_scan_joint" type="fixed" >
-      <origin xyz="0 0 0.09081" rpy="0 0 0" />
+      <origin xyz="0 0 0.0377" rpy="0 0 0" />
       <parent link="${name}_base_link" />
       <child link="${name}"/>
@@ -40,7 +45,7 @@
       </inertial>
       <visual>
-        <origin xyz="0 0 -0.09081" rpy="0 0 0" />
+        <origin xyz="0 0 -0.0377" />
         <geometry>
-          <mesh filename="package://husky_description/meshes/accessories/HDL32E_scan.dae" />
+          <mesh filename="package://velodyne_description/meshes/VLP16_scan.dae" />
         </geometry>
       </visual>
@@ -49,5 +54,5 @@
     <gazebo reference="${name}">
       <xacro:if value="${gpu}">
-        <sensor type="gpu_ray" name="${name}_VLP_16">
+          <sensor type="gpu_ray" name="${name}-VLP16">
           <pose>0 0 0 0 0 0</pose>
           <visualize>false</visualize>
@@ -64,10 +69,10 @@
                 <samples>${lasers}</samples>
                 <resolution>1</resolution>
-                <min_angle>-${15*M_PI/180.0}</min_angle>
-                <max_angle> ${15*M_PI/180.0}</max_angle>
+                <min_angle>-${15.0*M_PI/180.0}</min_angle>
+                <max_angle> ${15.0*M_PI/180.0}</max_angle>
               </vertical>
             </scan>
             <range>
-              <min>${min_range}</min>
+              <min>${collision_range}</min>
               <max>${max_range+1}</max>
               <resolution>0.001</resolution>
@@ -76,5 +81,5 @@
               <type>gaussian</type>
               <mean>0.0</mean>
-              <stddev>${noise}</stddev>
+              <stddev>0.0</stddev>
             </noise>
           </ray>

File: catkin_ws/src/husky/husky_description/urdf/husky.urdf.xacro (robot description, xacro)
@@ -137,4 +137,6 @@
     <plugin name="gazebo_ros_control" filename="libgazebo_ros_control.so">
       <robotNamespace>$(arg robot_namespace)</robotNamespace>
+      <robotSimType>gazebo_ros_control/DefaultRobotHWSim</robotSimType>
+      <legacyModeNS>true</legacyModeNS>
     </plugin>
   </gazebo>
@@ -171,10 +173,10 @@
   <xacro:include filename="$(arg urdf_extras)" />
   <xacro:include filename="$(find husky_description)/urdf/accessories/velodyne_lidar.urdf.xacro" />
-  <xacro:VLP16_lidar parent="top_plate_front_link" name="velodyne" topic="/velodyne_points" hz="8" samples="1800" min_range="0" max_range="50.0" min_angle="-3.14" max_angle="3.14" noise="0.008">
-    <origin xyz="0 0 0.04" rpy="0 0 0" />
+  <xacro:VLP16_lidar parent="top_plate_front_link" name="velodyne" topic="/velodyne_points" hz="8" samples="1800" min_range="0.5" max_range="50.0" min_angle="-3.14" max_angle="3.14" noise="0.008">
+    <origin xyz="-0.1 0 0.15" rpy="0 0 0" />
   </xacro:VLP16_lidar>
   <xacro:include filename="$(find husky_description)/urdf/accessories/camera.urdf.xacro" />
   <xacro:depth_camera parent="top_plate_front_link" name="camera" >
-    <origin xyz="0 0 0.02" rpy="0 0 1.57" />
+    <origin xyz="0 0.0 0.02" rpy="0 0 0" />
  </xacro:depth_camera>
 </robot>
